File: example_gerbers/basic/basic.kicad_pcb (KiCad board)
At the start: 2 copper layers, 10 x 15 mm, 0 parts

Commit message: Added postprocessing
Routing:
- net (no net): track 18.3 -> 14.3 mm
Changed lines of the file:
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@@
   (gr_rect (start 140 95) (end 150 110)
     (stroke (width 0.1) (type solid)) (fill none) (layer "Edge.Cuts"))
-  (segment (start 147.5 105.25) (end 147.5 101.25) (width 0.2) (layer "F.Cu") (net 0))
   (segment (start 145 98.171573) (end 145 96) (width 0.4) (layer "F.Cu") (net 0))
   (segment (start 145.585787 106.414213) (end 146.414214 105.585786) (width 0.4) (layer "F.Cu") (net 0))
