File: example_gerbers/basic/basic.kicad_pcb (KiCad board)
At the start: 2 copper layers, 9 x 14 mm, 6 parts

Commit message: Added support for multiple excitation
Parts:
- added SP3: Simulation-Port, antmicro-footprints:Simulation-Port, F.Cu at (146.5, 103.4)
Changed lines of the file:
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@@
   (net 1 "/MSL")
   (net 2 "GND")
+  (footprint "antmicro-footprints:Simulation-Port" (layer "F.Cu")
+    (at 146.5 103.4 180)
+    (attr board_only exclude_from_pos_files exclude_from_bom)
+    (fp_text reference "SP3" (at 0 1 180 unlocked) (layer "F.Fab")
+        (effects (font (size 1 1) (thickness 0.15)))
+    )
+    (fp_text value "Simulation-Port" (at 0 1 180 unlocked) (layer "F.Fab") hide
+        (effects (font (size 1 1) (thickness 0.15)))
+    )
+    (fp_text user "width = 0.4" (at 0 10) (layer "F.Fab") hide
+        (effects (font (size 1 1) (thickness 0.15)))
+    )
+    (fp_text user "${REFERENCE}" (at 0 2.5 180 unlocked) (layer "F.Fab") hide
+        (effects (font (size 1 1) (thickness 0.15)))
+    )
+    (fp_text user "stop_layer = 1" (at 0 8.5) (layer "F.Fab") hide
+        (effects (font (size 1 1) (thickness 0.15)))
+    )
+    (fp_text user "impedance = 50" (at 0 5.5) (layer "F.Fab") hide
+        (effects (font (size 1 1) (thickness 0.15)))
+    )
+    (fp_text user "start_layer = 0" (at 0 7) (layer "F.Fab") hide
+        (effects (font (size 1 1) (thickness 0.15)))
+    )
+    (fp_text user "excite = True" (at 0 11.5) (layer "F.Fab") hide
+        (effects (font (size 1 1) (thickness 0.15)))
+    )
+    (fp_text user "number = 1" (at 0 13) (layer "F.Fab") hide
+        (effects (font (size 1 1) (thickness 0.15)))
+    )
+    (fp_line (start -0.2 0) (end 0.2 0)
+      (stroke (width 0.12) (type solid)) (layer "Dwgs.User"))
+    (fp_line (start 0 -0.5) (end -0.1 -0.4)
+      (stroke (width 0.12) (type solid)) (layer "Dwgs.User"))
+    (fp_line (start 0 -0.5) (end 0.1 -0.4)
+      (stroke (width 0.12) (type solid)) (layer "Dwgs.User"))
+    (fp_line (start 0 0) (end 0 -0.5)
+      (stroke (width 0.12) (type solid)) (layer "Dwgs.User"))
+  )
   (footprint "antmicro-footprints:NetTie-2_SMD_Pad0.127mm" (layer "F.Cu")
     (at 147 112.4 90)
@@
         (effects (font (size 1 1) (thickness 0.15)))
     )
-    (fp_text user "width = 0.4" (at 0 10) (layer "F.Fab") hide
+    (fp_text user "number = 1" (at 0 13) (layer "F.Fab") hide
+        (effects (font (size 1 1) (thickness 0.15)))
+    )
+    (fp_text user "stop_layer = 1" (at 0 8.5) (layer "F.Fab") hide
+        (effects (font (size 1 1) (thickness 0.15)))
+    )
+    (fp_text user "excite = True" (at 0 11.5) (layer "F.Fab") hide
+        (effects (font (size 1 1) (thickness 0.15)))
+    )
+    (fp_text user "start_layer = 0" (at 0 7) (layer "F.Fab") hide
         (effects (font (size 1 1) (thickness 0.15)))
     )
@@
         (effects (font (size 1 1) (thickness 0.15)))
     )
-    (fp_text user "stop_layer = 1" (at 0 8.5) (layer "F.Fab") hide
+    (fp_text user "width = 0.4" (at 0 10) (layer "F.Fab") hide
         (effects (font (size 1 1) (thickness 0.15)))
     )
@@
         (effects (font (size 1 1) (thickness 0.15)))
     )
-    (fp_text user "start_layer = 0" (at 0 7) (layer "F.Fab") hide
-        (effects (font (size 1 1) (thickness 0.15)))
-    )
-    (fp_text user "excite = True" (at 0 11.5) (layer "F.Fab") hide
-        (effects (font (size 1 1) (thickness 0.15)))
-    )
-    (fp_text user "number = 1" (at 0 13) (layer "F.Fab") hide
-        (effects (font (size 1 1) (thickness 0.15)))
-    )

Commit message: Fix port name on PCB
Parts:
- SP1, SP2, SP3: value Simulation-Port -> Simulation_Port; footprint antmicro-footprints:Simulation-Port -> antmicro-footprints:Simulation_Port
- moved SP3 0.15 mm to (146.5, 103.2)
Changed lines of the file:
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@@
   (net 1 "/MSL")
   (net 2 "GND")
-  (footprint "antmicro-footprints:Simulation-Port" (layer "F.Cu")
-    (at 146.5 103.4 180)
-    (attr board_only exclude_from_pos_files exclude_from_bom)
-    (fp_text reference "SP3" (at 0 1 180 unlocked) (layer "F.Fab")
-        (effects (font (size 1 1) (thickness 0.15)))
-    )
-    (fp_text value "Simulation-Port" (at 0 1 180 unlocked) (layer "F.Fab") hide
-        (effects (font (size 1 1) (thickness 0.15)))
-    )
-    (fp_text user "width = 0.4" (at 0 10) (layer "F.Fab") hide
-        (effects (font (size 1 1) (thickness 0.15)))
-    )
-    (fp_text user "${REFERENCE}" (at 0 2.5 180 unlocked) (layer "F.Fab") hide
-        (effects (font (size 1 1) (thickness 0.15)))
-    )
-    (fp_text user "stop_layer = 1" (at 0 8.5) (layer "F.Fab") hide
-        (effects (font (size 1 1) (thickness 0.15)))
-    )
-    (fp_text user "impedance = 50" (at 0 5.5) (layer "F.Fab") hide
-        (effects (font (size 1 1) (thickness 0.15)))
-    )
-    (fp_text user "start_layer = 0" (at 0 7) (layer "F.Fab") hide
-        (effects (font (size 1 1) (thickness 0.15)))
-    )
-    (fp_text user "excite = True" (at 0 11.5) (layer "F.Fab") hide
-        (effects (font (size 1 1) (thickness 0.15)))
-    )
-    (fp_text user "number = 1" (at 0 13) (layer "F.Fab") hide
-        (effects (font (size 1 1) (thickness 0.15)))
-    )
-    (fp_line (start -0.2 0) (end 0.2 0)
-      (stroke (width 0.12) (type solid)) (layer "Dwgs.User"))
-    (fp_line (start 0 -0.5) (end -0.1 -0.4)
-      (stroke (width 0.12) (type solid)) (layer "Dwgs.User"))
-    (fp_line (start 0 -0.5) (end 0.1 -0.4)
-      (stroke (width 0.12) (type solid)) (layer "Dwgs.User"))
-    (fp_line (start 0 0) (end 0 -0.5)
-      (stroke (width 0.12) (type solid)) (layer "Dwgs.User"))
-  )
   (footprint "antmicro-footprints:NetTie-2_SMD_Pad0.127mm" (layer "F.Cu")
     (at 147 112.4 90)
@@
       (net 1 "/MSL") (pinfunction "2") (pintype "passive"))
   )
-  (footprint "antmicro-footprints:Simulation-Port" (layer "F.Cu")
-    (at 143 103.24 180)
+  (footprint "antmicro-footprints:Simulation_Port" (layer "F.Cu")
+    (at 146.5 103.25 180)
+    (descr "Place where port in the simulation should be located. Set it's reference to SPx, where x is port number")
     (attr board_only exclude_from_pos_files exclude_from_bom)
-    (fp_text reference "SP1" (at 0 1 180 unlocked) (layer "F.Fab")
+    (fp_text reference "SP3" (at 0 1 180 unlocked) (layer "F.Fab")
         (effects (font (size 1 1) (thickness 0.15)))
     )
-    (fp_text value "Simulation-Port" (at 0.1 0.64 180 unlocked) (layer "F.Fab") hide
+    (fp_text value "Simulation_Port" (at 0 5 180 unlocked) (layer "F.Fab") hide
         (effects (font (size 1 1) (thickness 0.15)))
     )
-    (fp_text user "stop_layer = 1" (at 0 8.5 180) (layer "F.Fab") hide
-        (effects (font (size 1 1) (thickness 0.15)))
-    )
-    (fp_text user "excite = True" (at 0 11.5 180) (layer "F.Fab") hide
-        (effects (font (size 1 1) (thickness 0.15)))
-    )
-    (fp_text user "impedance = 50" (at 0 5.5 180) (layer "F.Fab") hide
-        (effects (font (size 1 1) (thickness 0.15)))
-    )
-    (fp_text user "width = 0.4" (at 0 10 180) (layer "F.Fab") hide
-        (effects (font (size 1 1) (thickness 0.15)))
-    )
-    (fp_text user "number = 2" (at 0 13 180) (layer "F.Fab") hide
-        (effects (font (size 1 1) (thickness 0.15)))
-    )
-    (fp_text user "${REFERENCE}" (at -3.4 1.6 180 unlocked) (layer "F.Fab") hide
-        (effects (font (size 1 1) (thickness 0.15)))
-    )
-    (fp_text user "start_layer = 0" (at 0 7 180) (layer "F.Fab") hide
+    (fp_text user "{REFERENCE}" (at 0 3) (layer "F.Fab") hide
         (effects (font (size 1 1) (thickness 0.15)))
     )
     (fp_line (start -0.2 0) (end 0.2 0)
-      (stroke (width 0.12) (type solid)) (layer "Dwgs.User"))
-    (fp_line (start 0 -0.5) (end -0.1 -0.4)
-      (stroke (width 0.12) (type solid)) (layer "Dwgs.User"))
-    (fp_line (start 0 -0.5) (end 0.1 -0.4)
-      (stroke (width 0.12) (type solid)) (layer "Dwgs.User"))
+      (stroke (width 0.1) (type solid)) (layer "F.Fab"))
+    (fp_line (start 0 -0.5) (end -0.2 -0.3)
+      (stroke (width 0.1) (type solid)) (layer "F.Fab"))
+    (fp_line (start 0 -0.5) (end 0.2 -0.3)
+      (stroke (width 0.1) (type solid)) (layer "F.Fab"))
     (fp_line (start 0 0) (end 0 -0.5)
-      (stroke (width 0.12) (type solid)) (layer "Dwgs.User"))
+      (stroke (width 0.1) (type solid)) (layer "F.Fab"))
+  )
+  (footprint "antmicro-footprints:Simulation_Port" (layer "F.Cu")
+    (at 147 112.75)
+    (descr "Place where port in the simulation should be located. Set it's reference to SPx, where x is port number")
+    (attr board_only exclude_from_pos_files exclude_from_bom)
+    (fp_text reference "SP2" (at 0 1 unlocked) (layer "F.Fab")
+        (effects (font (size 1 1) (thickness 0.15)))
+    )
+    (fp_text value "Simulation_Port" (at 0 5 unlocked) (layer "F.Fab") hide
+        (effects (font (size 1 1) (thickness 0.15)))
+    )
+    (fp_text user "{REFERENCE}" (at 0 3) (layer "F.Fab") hide
+        (effects (font (size 1 1) (thickness 0.15)))
+    )
+    (fp_line (start -0.2 0) (end 0.2 0)
+      (stroke (width 0.1) (type solid)) (layer "F.Fab"))
+    (fp_line (start 0 -0.5) (end -0.2 -0.3)
+      (stroke (width 0.1) (type solid)) (layer "F.Fab"))
+    (fp_line (start 0 -0.5) (end 0.2 -0.3)
+      (stroke (width 0.1) (type solid)) (layer "F.Fab"))
+    (fp_line (start 0 0) (end 0 -0.5)
+      (stroke (width 0.1) (type solid)) (layer "F.Fab"))
   )
   (footprint "antmicro-footprints:NetTie-2_SMD_Pad0.127mm" (layer "F.Cu")
@@
       (net 1 "/MSL") (pinfunction "2") (pintype "passive"))
   )
-  (footprint "antmicro-footprints:Simulation-Port" (layer "F.Cu")
-    (at 147 112.7)
+  (footprint "antmicro-footprints:Simulation_Port" (layer "F.Cu")
+    (at 143 103.25 180)
+    (descr "Place where port in the simulation should be located. Set it's reference to SPx, where x is port number")
     (attr board_only exclude_from_pos_files exclude_from_bom)
-    (fp_text reference "SP2" (at 0 1 unlocked) (layer "F.Fab")
+    (fp_text reference "SP1" (at 0 1 180 unlocked) (layer "F.Fab")
         (effects (font (size 1 1) (thickness 0.15)))
     )
-    (fp_text value "Simulation-Port" (at 0 1 unlocked) (layer "F.Fab") hide
+    (fp_text value "Simulation_Port" (at 0 5 180 unlocked) (layer "F.Fab") hide
         (effects (font (size 1 1) (thickness 0.15)))
     )
-    (fp_text user "number = 1" (at 0 13) (layer "F.Fab") hide
-        (effects (font (size 1 1) (thickness 0.15)))
-    )
-    (fp_text user "stop_layer = 1" (at 0 8.5) (layer "F.Fab") hide
-        (effects (font (size 1 1) (thickness 0.15)))
-    )
-    (fp_text user "excite = True" (at 0 11.5) (layer "F.Fab") hide
-        (effects (font (size 1 1) (thickness 0.15)))
-    )
-    (fp_text user "start_layer = 0" (at 0 7) (layer "F.Fab") hide
-        (effects (font (size 1 1) (thickness 0.15)))
-    )
-    (fp_text user "${REFERENCE}" (at 0 2.5 unlocked) (layer "F.Fab") hide
-        (effects (font (size 1 1) (thickness 0.15)))
-    )
-    (fp_text user "width = 0.4" (at 0 10) (layer "F.Fab") hide
-        (effects (font (size 1 1) (thickness 0.15)))
-    )
-    (fp_text user "impedance = 50" (at 0 5.5) (layer "F.Fab") hide
+    (fp_text user "{REFERENCE}" (at 0 3) (layer "F.Fab") hide
         (effects (font (size 1 1) (thickness 0.15)))
     )
     (fp_line (start -0.2 0) (end 0.2 0)
-      (stroke (width 0.12) (type solid)) (layer "Dwgs.User"))
-    (fp_line (start 0 -0.5) (end -0.1 -0.4)
-      (stroke (width 0.12) (type solid)) (layer "Dwgs.User"))
-    (fp_line (start 0 -0.5) (end 0.1 -0.4)
-      (stroke (width 0.12) (type solid)) (layer "Dwgs.User"))
+      (stroke (width 0.1) (type solid)) (layer "F.Fab"))
+    (fp_line (start 0 -0.5) (end -0.2 -0.3)
+      (stroke (width 0.1) (type solid)) (layer "F.Fab"))
+    (fp_line (start 0 -0.5) (end 0.2 -0.3)
+      (stroke (width 0.1) (type solid)) (layer "F.Fab"))
     (fp_line (start 0 0) (end 0 -0.5)
-      (stroke (width 0.12) (type solid)) (layer "Dwgs.User"))
+      (stroke (width 0.1) (type solid)) (layer "F.Fab"))
   )
   (footprint "antmicro-footprints:NetTie-2_SMD_Pad0.127mm" (layer "B.Cu")
