File: example_gerbers/real/real.kicad_pcb (KiCad board)
At the start: 2 copper layers, 4.2 x 14.7 mm, 2 parts

Commit message: Working real test case
Parts:
- added TP1: TP_0.75mm_SMD, antmicro-footprints:TP_SMD_0.75mm, F.Cu at (148.8, 95.9)
Routing:
- net /net: track 0.00 -> 21.0 mm
- net (no net): track 21.0 -> 0.00 mm
