File: example_gerbers/differential/differential.kicad_pcb (KiCad board)
At the start: 2 copper layers, 4 x 16 mm, 8 parts

Commit message: Change port numbering in differential pair example
Parts:
- renumbered SP1 to SP0, SP2 to SP1, SP3 to SP2, SP4 to SP3
