File: examples/job-simulation-part/jetson-orin-baseboard.kicad_pcb (KiCad board)
At the start: 8 copper layers, 12.9 x 31.2 mm, 22 parts, among them Q2 PJE138K, U45 TPD4E05U06QDQARQ1

Commit message: Update job example
Parts:
- removed R214, R220: R_499R_0402, jetson-orin-baseboard-footprints:R_0402_1005Metric
Routing:
- net GND: track 278.3 -> 271.7 mm, vias 5 -> 3
Changed lines of the file:
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@@
       (stroke (width 0.1) (type solid)) (layer "F.Fab"))
-  )
-  (footprint "jetson-orin-baseboard-footprints:R_0402_1005Metric" (layer "F.Cu")
-    (at 91.02 103.28 -135)
-    (descr "Resistor SMD 0402")
-    (tags "resistor SMD 0402")
-    (property "Author" "Antmicro")
-    (property "License" "Apache-2.0")
-    (property "MPN" "CR0402-FX-4990GLF")
-    (property "Manufacturer" "Vishay")
-    (property "Sheetfile" "hdmi.kicad_sch")
-    (property "Sheetname" "HDMI")
-    (property "Tolerance" "1%")
-    (property "Val" "499R")
-    (attr smd)
-    (fp_text reference "R220" (at 0.707107 -1.470782 -135) (layer "F.SilkS")
-        (effects (font (size 0.7 0.7) (thickness 0.15)) (justify left bottom))
-    )
-    (fp_text value "R_499R_0402" (at -0.378302 1.113693 -135) (layer "F.Fab")
-        (effects (font (size 0.7 0.7) (thickness 0.15)) (justify left bottom))
-    )
-    (fp_text user "${REFERENCE}" (at -0.95 3.168 -135) (layer "F.Fab") hide
-        (effects (font (size 0.7 0.7) (thickness 0.15)) (justify left bottom))
-    )
-    (fp_text user "License: Apache-2.0" (at -0.949999 5.169 -135) (layer "F.Fab") hide
-        (effects (font (size 0.7 0.7) (thickness 0.15)) (justify left bottom))
-    )
-    (fp_text user "Author: Antmicro" (at -0.95 4.169 -135) (layer "F.Fab") hide
-        (effects (font (size 0.7 0.7) (thickness 0.15)) (justify left bottom))
-    )
-    (fp_rect (start -0.93 -0.47) (end 0.93 0.47)
-      (stroke (width 0.05) (type solid)) (fill none) (layer "F.CrtYd"))
-    (fp_rect (start -0.5 -0.25) (end 0.5 0.25)
-      (stroke (width 0.15) (type solid)) (fill none) (layer "F.Fab"))
-    (fp_rect (start -0.5 -0.25) (end 0.5 0.25)
-      (stroke (width 0.1) (type solid)) (fill none) (layer "User.5"))
-    (fp_line (start -0.5 0.248) (end -0.5 -0.25)
-      (stroke (width 0.02) (type solid)) (layer "User.9"))
-    (fp_line (start -0.25 -0.25) (end -0.5 -0.25)
-      (stroke (width 0.02) (type solid)) (layer "User.9"))
-    (fp_line (start -0.25 0.248) (end -0.5 0.248)
-      (stroke (width 0.02) (type solid)) (layer "User.9"))
-    (fp_line (start -0.25 0.248) (end -0.25 -0.25)
-      (stroke (width 0.02) (type solid)) (layer "User.9"))
-    (fp_line (start 0.248 -0.25) (end 0.248 0.248)
-      (stroke (width 0.02) (type solid)) (layer "User.9"))
-    (fp_line (start 0.248 -0.232) (end -0.25 -0.232)
-      (stroke (width 0.02) (type solid)) (layer "User.9"))
-    (fp_line (start 0.248 0.23) (end -0.25 0.23)
-      (stroke (width 0.02) (type solid)) (layer "User.9"))
-    (fp_line (start 0.248 0.248) (end 0.498 0.248)
-      (stroke (width 0.02) (type solid)) (layer "User.9"))
-    (fp_line (start 0.498 -0.25) (end 0.248 -0.25)
-      (stroke (width 0.02) (type solid)) (layer "User.9"))
-    (fp_line (start 0.498 0.248) (end 0.498 -0.25)
-      (stroke (width 0.02) (type solid)) (layer "User.9"))
-    (pad "1" smd roundrect (at -0.485 0 225) (size 0.59 0.64) (layers "F.Cu" "F.Paste" "F.Mask") (roundrect_rratio 0.25)
-      (net 1 "GND") (pintype "passive"))
-    (pad "2" smd roundrect (at 0.485 0 225) (size 0.59 0.64) (layers "F.Cu" "F.Paste" "F.Mask") (roundrect_rratio 0.25)
-      (net 363 "/HDMI/HDMI_D0_P") (pintype "passive"))
-    (model "${KIPRJMOD}/lib/3d-models/R_0402_1005Metric.step"
-      (offset (xyz 0 0 -0.01))
-      (scale (xyz 1 1 1))
-      (rotate (xyz 0 0 0))
-    )
   )
   (footprint "antmicro-footprints:Simulation_Port" (layer "F.Cu")
@@
     (fp_line (start 0 0) (end 0 -0.5)
       (stroke (width 0.1) (type solid)) (layer "F.Fab"))
-  )
-  (footprint "jetson-orin-baseboard-footprints:R_0402_1005Metric" (layer "F.Cu")
-    (at 89.7 104.6 45)
-    (descr "Resistor SMD 0402")
-    (tags "resistor SMD 0402")
-    (property "Author" "Antmicro")
-    (property "License" "Apache-2.0")
-    (property "MPN" "CR0402-FX-4990GLF")
-    (property "Manufacturer" "Vishay")
-    (property "Sheetfile" "hdmi.kicad_sch")
-    (property "Sheetname" "HDMI")
-    (property "Tolerance" "1%")
-    (property "Val" "499R")
-    (attr smd)
-    (fp_text reference "R214" (at -1.704127 1.477853 45) (layer "F.SilkS")
-        (effects (font (size 0.7 0.7) (thickness 0.15)) (justify left bottom))
-    )
-    (fp_text value "R_499R_0402" (at 0 1.399999 45) (layer "F.Fab")
-        (effects (font (size 0.7 0.7) (thickness 0.15)) (justify left bottom))
-    )
-    (fp_text user "Author: Antmicro" (at -0.95 4.169 45) (layer "F.Fab") hide
-        (effects (font (size 0.7 0.7) (thickness 0.15)) (justify left bottom))
-    )
-    (fp_text user "${REFERENCE}" (at -0.95 3.168 45) (layer "F.Fab") hide
-        (effects (font (size 0.7 0.7) (thickness 0.15)) (justify left bottom))
-    )
-    (fp_text user "License: Apache-2.0" (at -0.949999 5.169 45) (layer "F.Fab") hide
-        (effects (font (size 0.7 0.7) (thickness 0.15)) (justify left bottom))
-    )
-    (fp_rect (start -0.93 -0.47) (end 0.93 0.47)
-      (stroke (width 0.05) (type solid)) (fill none) (layer "F.CrtYd"))
-    (fp_rect (start -0.5 -0.25) (end 0.5 0.25)
-      (stroke (width 0.15) (type solid)) (fill none) (layer "F.Fab"))
-    (fp_rect (start -0.5 -0.25) (end 0.5 0.25)
-      (stroke (width 0.1) (type solid)) (fill none) (layer "User.5"))
-    (fp_line (start -0.5 0.248) (end -0.5 -0.25)
-      (stroke (width 0.02) (type solid)) (layer "User.9"))
-    (fp_line (start -0.25 -0.25) (end -0.5 -0.25)
-      (stroke (width 0.02) (type solid)) (layer "User.9"))
-    (fp_line (start -0.25 0.248) (end -0.5 0.248)
-      (stroke (width 0.02) (type solid)) (layer "User.9"))
-    (fp_line (start -0.25 0.248) (end -0.25 -0.25)
-      (stroke (width 0.02) (type solid)) (layer "User.9"))
-    (fp_line (start 0.248 -0.25) (end 0.248 0.248)
-      (stroke (width 0.02) (type solid)) (layer "User.9"))
-    (fp_line (start 0.248 -0.232) (end -0.25 -0.232)
-      (stroke (width 0.02) (type solid)) (layer "User.9"))
-    (fp_line (start 0.248 0.23) (end -0.25 0.23)
-      (stroke (width 0.02) (type solid)) (layer "User.9"))
-    (fp_line (start 0.248 0.248) (end 0.498 0.248)
-      (stroke (width 0.02) (type solid)) (layer "User.9"))
-    (fp_line (start 0.498 -0.25) (end 0.248 -0.25)
-      (stroke (width 0.02) (type solid)) (layer "User.9"))
-    (fp_line (start 0.498 0.248) (end 0.498 -0.25)
-      (stroke (width 0.02) (type solid)) (layer "User.9"))
-    (pad "1" smd roundrect (at -0.485 0 45) (size 0.59 0.64) (layers "F.Cu" "F.Paste" "F.Mask") (roundrect_rratio 0.25)
-      (net 1 "GND") (pintype "passive"))
-    (pad "2" smd roundrect (at 0.485 0 45) (size 0.59 0.64) (layers "F.Cu" "F.Paste" "F.Mask") (roundrect_rratio 0.25)
-      (net 357 "/HDMI/HDMI_D0_N") (pintype "passive"))
-    (model "${KIPRJMOD}/lib/3d-models/R_0402_1005Metric.step"
-      (offset (xyz 0 0 -0.01))
-      (scale (xyz 1 1 1))
-      (rotate (xyz 0 0 0))
-    )
   )
   (footprint "jetson-orin-baseboard-footprints:R_0402_1005Metric" (layer "F.Cu")
@@
   (segment (start 93.625 120.825) (end 93.625 120.285) (width 0.2) (layer "F.Cu") (net 1))
   (segment (start 93.625 119.515) (end 93.625 120.285) (width 0.2) (layer "F.Cu") (net 1))
-  (segment (start 88.8 100.2) (end 88.15 100.2) (width 0.125) (layer "F.Cu") (net 1))
-  (segment (start 88.95 103.7) (end 89.2 103.45) (width 0.125) (layer "F.Cu") (net 1))
-  (segment (start 89.357053 104.942947) (end 89.357053 104.877053) (width 0.125) (layer "F.Cu") (net 1))
   (segment (start 93.95 121.15) (end 93.625 120.825) (width 0.2) (layer "F.Cu") (net 1))
-  (segment (start 90.95 102.3) (end 90.94 102.31) (width 0.15) (layer "F.Cu") (net 1))
-  (segment (start 89.2 100.6) (end 88.8 100.2) (width 0.125) (layer "F.Cu") (net 1))
   (segment (start 91.45 102.35) (end 91.75 102.35) (width 0.125) (layer "F.Cu") (net 1))
-  (segment (start 89.2 103.45) (end 89.2 100.6) (width 0.125) (layer "F.Cu") (net 1))
-  (segment (start 91.307053 102.937053) (end 91.362947 102.937053) (width 0.15) (layer "F.Cu") (net 1))
-  (segment (start 90.94 102.31) (end 90.94 102.57) (width 0.15) (layer "F.Cu") (net 1))
-  (segment (start 90.94 102.57) (end 91.307053 102.937053) (width 0.15) (layer "F.Cu") (net 1))
-  (segment (start 89.357053 104.877053) (end 88.95 104.47) (width 0.125) (layer "F.Cu") (net 1))
-  (segment (start 88.95 104.47) (end 88.95 103.7) (width 0.125) (layer "F.Cu") (net 1))
   (via (at 91.45 102.35) (size 0.45) (drill 0.1) (layers "F.Cu" "B.Cu") (remove_unused_layers) (keep_end_layers) (zone_layer_connections "In1.Cu" "In2.Cu" "In4.Cu" "In6.Cu") (net 1))
   (via (at 91.75 108.8) (size 0.45) (drill 0.1) (layers "F.Cu" "B.Cu") (remove_unused_layers) (keep_end_layers) (zone_layer_connections "In1.Cu" "In2.Cu" "In4.Cu" "In6.Cu") (net 1))
   (via (at 94.962501 117.706675) (size 0.45) (drill 0.1) (layers "F.Cu" "B.Cu") (remove_unused_layers) (keep_end_layers) (free) (zone_layer_connections "In1.Cu" "In6.Cu") (net 1))
-  (via (at 89.2 103.45) (size 0.45) (drill 0.1) (layers "F.Cu" "B.Cu") (remove_unused_layers) (keep_end_layers) (zone_layer_connections "In1.Cu" "In2.Cu" "In4.Cu" "In6.Cu") (net 1))
-  (via (at 90.95 102.3) (size 0.45) (drill 0.1) (layers "F.Cu" "B.Cu") (remove_unused_layers) (keep_end_layers) (zone_layer_connections "In1.Cu" "In2.Cu" "In4.Cu" "In6.Cu") (net 1))
   (segment (start 90.35 102.3) (end 89.2 103.45) (width 0.125) (layer "In5.Cu") (net 1))
   (segment (start 92.09 101.16) (end 90.95 102.3) (width 0.125) (layer "In5.Cu") (net 1))
